File: Fast_Passive_Probe_20x.kicad_sch (KiCad schematic)
At the start: 7 parts, among them J1 Conn_Coaxial, J2 Conn_Coaxial

Commit message: testy
dodano screeny testow wygenerowano pdfa schematu
Other:
- note added: "50 Ohm termination"
- note added: "SCOPE"
- note added: "or 0 Ohm"
- title: (none) -> Fast_Passive_Probe_20x
- moved on the sheet: C1, H3, H4, J1, J2, R1, R2
